Commit message: added "gripper_scups_link" in the urdf for the rotations related with the suction cups

File: harvest_hardware/ur5e_custom_hardware/urdf/gripper.urdf.xacro (robot description, xacro)
@@ -2,4 +2,16 @@
 <robot xmlns:xacro="http://www.ros.org/wiki/xacro" >
     <xacro:macro name="gripper_macro">
+    <joint name="gripper_scups_joint" type="fixed">
+        <parent link="gripper_link"/>
+        <child link="gripper_scups_link"/>
+        <origin xyz="0.00 0.00 -0.02" rpy="0 0 -3.1416"/>
+    </joint>
+    <link name="gripper_scups_link">
+        <!-- <collision>
+            <geometry>
+                <box size="0.08 0.05 0.01"/>
+            </geometry>
+        </collision> -->
+    </link>
     <joint name="gripper_palm_camera_joint" type="fixed">
         <parent link="gripper_link"/>

Commit message: (1) included 'release_apple' service (2) added 'scups_link' in urdf

File: harvest_hardware/ur5e_custom_hardware/urdf/gripper.urdf.xacro (robot description, xacro)
@@ -5,12 +5,15 @@
         <parent link="gripper_link"/>
         <child link="gripper_scups_link"/>
-        <origin xyz="0.00 0.00 -0.02" rpy="0 0 -3.1416"/>
+        <origin xyz="0.00 0.00 -0.02" rpy="0 0 -2.618"/>
     </joint>
     <link name="gripper_scups_link">
-        <!-- <collision>
+        <visual>
             <geometry>
-                <box size="0.08 0.05 0.01"/>
+                <box size="0.01 0.01 0.01"/>
             </geometry>
-        </collision> -->
+            <material name="green">
+                <color rgba="0 1 0 1"/>
+            </material>
+        </visual>
     </link>
     <joint name="gripper_palm_camera_joint" type="fixed">

Commit message: Changes during Prosser'24 end of day1

File: harvest_hardware/ur5e_custom_hardware/urdf/gripper.urdf.xacro (robot description, xacro)
@@ -26,4 +26,5 @@
         <child link="gripper_top_camera_link"/>
         <origin xyz="0.00 -.072 -0.0865" rpy="0 0 0"/>
+        <!-- <origin xyz="0.009525 -.08255 -0.0445" rpy="0 0 0"/> -->
     </joint>
     <link name="gripper_top_camera_link">

Commit message: filtering point cloud based on apple locations. modified camera intrinsics and mount location

File: harvest_hardware/ur5e_custom_hardware/urdf/gripper.urdf.xacro (robot description, xacro)
@@ -1,67 +1,85 @@
 <?xml version="1.0"?>
-<robot xmlns:xacro="http://www.ros.org/wiki/xacro" >
+<robot xmlns:xacro="http://www.ros.org/wiki/xacro">
     <xacro:macro name="gripper_macro">
-    <joint name="gripper_scups_joint" type="fixed">
-        <parent link="gripper_link"/>
-        <child link="gripper_scups_link"/>
-        <origin xyz="0.00 0.00 -0.02" rpy="0 0 -2.618"/>
-    </joint>
-    <link name="gripper_scups_link">
-        <visual>
-            <geometry>
-                <box size="0.01 0.01 0.01"/>
-            </geometry>
-            <material name="green">
-                <color rgba="0 1 0 1"/>
-            </material>
-        </visual>
-    </link>
-    <joint name="gripper_palm_camera_joint" type="fixed">
-        <parent link="gripper_link"/>
-        <child link="gripper_palm_camera_optical_link"/>
-        <origin xyz="0.00 0 -0.05" rpy="0 0 0"/>
-    </joint>
-    <joint name="gripper_top_camera_joint" type="fixed">
-        <parent link="gripper_link"/>
-        <child link="gripper_top_camera_link"/>
-        <origin xyz="0.00 -.072 -0.0865" rpy="0 0 0"/>
-        <!-- <origin xyz="0.009525 -.08255 -0.0445" rpy="0 0 0"/> -->
-    </joint>
-    <link name="gripper_top_camera_link">
-        <!-- <collision>
+        <joint name="gripper_scups_joint" type="fixed">
+            <parent link="gripper_link" />
+            <child link="gripper_scups_link" />
+            <origin xyz="0.00 0.00 -0.02" rpy="0 0 -2.618" />
+        </joint>
+        <link name="gripper_scups_link">
+            <visual>
+                <geometry>
+                    <box size="0.01 0.01 0.01" />
+                </geometry>
+                <material name="green">
+                    <color rgba="0 1 0 1" />
+                </material>
+            </visual>
+        </link>
+        <joint name="gripper_palm_camera_joint" type="fixed">
+            <parent link="gripper_link" />
+            <child link="gripper_palm_camera_optical_link" />
+            <origin xyz="0.00 0 -0.05" rpy="0 0 0" />
+        </joint>
+        <joint name="gripper_top_camera_joint" type="fixed">
+            <parent link="gripper_link" />
+            <child link="gripper_top_camera_link" />
+            <origin xyz="0.00 -.072 -0.0865" rpy="0 0 0" />
+            <!-- <origin xyz="0.009525 -.08255 -0.0445" rpy="0 0 0"/> -->
+        </joint>
+        <link name="gripper_top_camera_link">
+            <!-- <collision>
             <geometry>
                 <box size="0.08 0.05 0.01"/>
             </geometry>
         </collision> -->
-    </link>
-    <link name="gripper_palm_camera_optical_link">
-        <visual>
-            <geometry>
-                <box size="0.03 0.03 0.01"/>
-            </geometry>
-            <material name="green">
-                <color rgba="0 1 0 1"/>
-            </material>
-        </visual>
-    </link>
-    <link name="gripper_link">
-        <collision>
-            <origin xyz="0.00 0 -0.105" rpy="0 0 0"/>
-            <geometry>
-                <box size="0.12 0.12 0.2"/>
-            </geometry>
-        </collision>
-        <visual>
-            <origin xyz="0.085 0 -0.2" rpy="0 0 3.14"/>
-            <geometry>
-                <mesh filename="package://ur5e_custom_hardware/meshes/03_mk3_full_assembly_coarse.STL" scale="0.001 0.001 0.001"/>
-            </geometry>
-        </visual>
-    </link>
-    <xacro:arg name="use_nominal_extrinsics" default="false" />
+        </link>
+        <link name="gripper_palm_camera_optical_link">
+            <visual>
+                <geometry>
+                    <box size="0.03 0.03 0.01" />
+                </geometry>
+                <material name="green">
+                    <color rgba="0 1 0 1" />
+                </material>
+            </visual>
+        </link>
+        <link name="gripper_link">
+            <collision>
+                <origin xyz="0.00 0 -0.105" rpy="0 0 0" />
+                <geometry>
+                    <box size="0.12 0.12 0.2" />
+                </geometry>
+            </collision>
+            <visual>
+                <origin xyz="0.085 0 -0.2" rpy="0 0 3.14" />
+                <geometry>
+                    <mesh
+                        filename="package://ur5e_custom_hardware/meshes/03_mk3_full_assembly_coarse.STL"
+                        scale="0.001 0.001 0.001" />
+                </geometry>
+            </visual>
+        </link>
+        <joint name="camera_joint" type="fixed">
+            <parent link="gripper_link" />
+            <child link="camera_link" />
+            <origin xyz="0.00 0.00 -0.5" rpy="0 0 0" />
+        </joint>
+        <link name="camera_link">
+            <visual>
+                <geometry>
+                    <box size="0.03 0.03 0.01" />
+                </geometry>
+                <material name="green">
+                    <color rgba="0 1 0 1" />
+                </material>
+            </visual>
+        </link>
+        <!-- <xacro:arg name="use_nominal_extrinsics" default="false" />
     <xacro:include filename="$(find realsense2_description)/urdf/_d435i.urdf.xacro"/>
-    <xacro:sensor_d435i parent="gripper_top_camera_link" use_nominal_extrinsics="$(arg use_nominal_extrinsics)">
-      <origin xyz="0 0 0" rpy="0 -1.571 1.571"/>
-    </xacro:sensor_d435i>
-</xacro:macro>
+    <xacro:sensor_d435i parent="gripper_top_camera_link" use_nominal_extrinsics="$(arg
+        use_nominal_extrinsics)">
+      <origin xyz="0 0 -0.5" rpy="0 -1.571 1.571"/>
+    </xacro:sensor_d435i> -->
+    </xacro:macro>
 </robot>

File: harvest_hardware/ur5e_custom_hardware/urdf/ur_gripper.urdf.xacro (robot description, xacro)
@@ -46,5 +46,6 @@
    <xacro:arg name="simulation_controllers" default="" />
    <!-- initial position for simulations (Fake Hardware, Gazebo, Ignition) -->
-   <xacro:arg name="initial_positions_file" default="$(find ur_description)/config/initial_positions.yaml"/>
+   <!-- <xacro:arg name="initial_positions_file" default="$(find ur_description)/config/initial_positions.yaml"/> -->
+   <xacro:arg name="initial_positions_file" default="$(find ur_description)/config/initial_positions_marcus.yaml"/>
    <!-- convert to property to use substitution in function -->
    <xacro:property name="initial_positions_file" default="$(arg initial_positions_file)"/>

Commit message: updated camera intrinsics for microsoft azure kinect. implmented go-to-pose pipeline using RRT-star for ur5

File: harvest_hardware/ur5e_custom_hardware/urdf/gripper.urdf.xacro (robot description, xacro)
@@ -62,7 +62,9 @@
         </link>
         <joint name="camera_joint" type="fixed">
-            <parent link="gripper_link" />
+            <!-- <parent link="gripper_link" /> -->
+            <parent link="base_link" />
             <child link="camera_link" />
-            <origin xyz="0.00 0.00 -0.5" rpy="0 0 0" />
+            <!-- <origin xyz="0.00 0.00 0.5" rpy="0 0 0" /> -->
+            <origin xyz="0.00 0.00 0.5" rpy="-1.57079 0 0" />
         </joint>
         <link name="camera_link">

Commit message: converting point cloud visual from rgb to bgr, removed green camera link visual, made a short results processing script

File: harvest_hardware/ur5e_custom_hardware/urdf/gripper.urdf.xacro (robot description, xacro)
@@ -69,5 +69,5 @@
         </joint>
         <link name="camera_link">
-            <visual>
+            <!-- <visual>
                 <geometry>
                     <box size="0.03 0.03 0.01" />
@@ -76,5 +76,5 @@
                     <color rgba="0 1 0 1" />
                 </material>
-            </visual>
+            </visual> -->
         </link>
         <!-- <xacro:arg name="use_nominal_extrinsics" default="false" />

Commit message: added camera intrinsics for voxelization, image generation, updated moveit ik solver to trac-ik

File: harvest_hardware/ur5e_custom_hardware/urdf/gripper.urdf.xacro (robot description, xacro)
@@ -59,4 +59,7 @@
                         scale="0.001 0.001 0.001" />
                 </geometry>
+                <material name="ur5_blue">
+                    <color rgba="0.45 0.62 0.9 1" />
+                </material>
             </visual>
         </link>
@@ -66,5 +69,5 @@
             <child link="camera_link" />
             <!-- <origin xyz="0.00 0.00 0.5" rpy="0 0 0" /> -->
-            <origin xyz="0.00 0.00 0.5" rpy="-1.57079 0 0" />
+            <origin xyz="0.00 -0.1 0.5" rpy="-1.57079 0 0" />
         </joint>
         <link name="camera_link">
