Commit message: adds amgia to main launch. removes source install of realsense

File: harvest_hardware/robot_custom_hardware/urdf/amiga.urdf.xacro (robot description, xacro)
@@ -18,8 +18,6 @@
     <xacro:property name="amiga_collision_box2_y" value='0.25' />
     <xacro:property name="amiga_collision_box2_z" value='0.25' />
-    <!-- <xacro:property name="amiga_tool0_mount_rotation" value="0.0 0.0 -${pi / 4 + pi}"/> -->
-    <xacro:property name="amiga_tool0_mount_rotation" value="0.0 0.0 0.0"/>
-    <!-- <xacro:property name="amiga_tool0_mount_position" value="-0.12825037 0.323256 0.99810607"/> -->
-    <xacro:property name="amiga_tool0_mount_position" value="-0.225 0.323256 ${0.99810607+0.1}"/>
+    <xacro:property name="amiga_tool0_mount_rotation" value="0.0 0.0 ${pi / 4}"/>
+    <xacro:property name="amiga_tool0_mount_position" value="-0.225 0.323256 1.0"/>
     <!-- ================== -->
     <!--       Links        -->
@@ -34,5 +32,5 @@
             <material name="LightLightGrey"/>
         </visual>
-        <collision>
+        <!-- <collision>
             <origin rpy="0.0 0.0 0.0" xyz="0.0 0.0 ${amiga_collision_box0_z / 2}"/>
             <geometry>
@@ -50,4 +48,10 @@
             <geometry>
                 <box size="${amiga_collision_box2_x} ${amiga_collision_box2_y} ${amiga_collision_box2_z}" />
+            </geometry>
+        </collision> -->
+        <collision>
+            <origin rpy="0.0 0.0 0.0" xyz="0.0 0.0 0.0"/>
+            <geometry>
+                <mesh filename="${mesh_base_path}base_mounts/frame_on_amiga_v2_simplified.stl"/>
             </geometry>
         </collision>

File: harvest_hardware/robot_custom_hardware/urdf/amiga_ur_gripper.urdf.xacro (robot description, xacro)
@@ -33,10 +33,11 @@
   <xacro:arg name="sim_ignition" default="false"/>
   <xacro:arg name="simulation_controllers" default=""/>
-  <!-- initial positions in your pkg -->
   <xacro:arg name="initial_positions_file" default="$(find robot_custom_hardware)/config/initial_positions.yaml"/>
   <xacro:property name="initial_positions_file" default="$(arg initial_positions_file)"/>
+  <!-- Amiga args -->
+  <xacro:arg name="amiga_prefix" default="amiga__"/>
   <!-- Realsense args -->
-  <xacro:arg name="use_nominal_extrinsics" default="false" />
-  <!-- CRITICAL: define the four args with the names the UR macro expects -->
+  <xacro:arg name="use_nominal_extrinsics" default="true" />
+  <!-- Define the four args with the names the UR macro expects -->
   <xacro:arg name="joint_limit_params" default="$(find robot_custom_hardware)/config/ur5e/joint_limits.yaml"/>
   <xacro:arg name="kinematics_params"  default="$(find robot_custom_hardware)/config/ur5e/default_kinematics.yaml"/>
@@ -47,10 +48,9 @@
   <xacro:include filename="$(find ur_description)/urdf/ur_macro.xacro"/>
   <xacro:include filename="$(find robot_custom_hardware)/urdf/gripper.urdf.xacro"/>
-  <xacro:include filename="$(find realsense2_description)/urdf/_d435i.urdf.xacro"/>
+  <xacro:include filename="$(find robot_custom_hardware)/urdf/_d435i.urdf.xacro"/>
   <!-- define world exactly once -->
   <link name="world"/>
   <!-- Instantiate Amiga, attached to world.
-       NOTE: your amiga macro signature requires mesh_base_path;
-       if it actually uses $(robot_custom_hardware) inside, define a property it expects. -->
+       NOTE: your amiga macro signature requires mesh_base_path -->
   <xacro:property name="robot_custom_hardware" value="package://robot_custom_hardware/"/>
   <xacro:amiga_macro amiga_prefix="$(arg amiga_prefix)" amiga_parent="world" mesh_base_path="package://robot_custom_hardware/meshes/"/>
@@ -101,6 +101,17 @@
   </joint>
   <xacro:gripper_macro/>
-  <xacro:sensor_d435i parent="base_link" use_nominal_extrinsics="$(arg use_nominal_extrinsics)">
-    <origin xyz="0.47625 -0.4907 0.4667" rpy="0 0 1.8852"/>
+  <!-- Realsense for apple locations -->
+  <xacro:sensor_d435i
+    parent="$(arg amiga_prefix)base"
+    prefix="mast_"
+    use_nominal_extrinsics="$(arg use_nominal_extrinsics)">
+    <origin xyz="0.3 -0.2 1.4667" rpy="0 0 1.8852"/>
+  </xacro:sensor_d435i>
+  <!-- Realsense for trunk detections -->
+  <xacro:sensor_d435i
+    parent="$(arg amiga_prefix)base"
+    prefix="base_"
+    use_nominal_extrinsics="$(arg use_nominal_extrinsics)">
+    <origin xyz="0.0 0.385 0.5588" rpy="0 0 1.57"/>
   </xacro:sensor_d435i>
 </robot>

File: harvest_hardware/robot_custom_hardware/urdf/gripper.urdf.xacro (robot description, xacro)
@@ -8,5 +8,5 @@
         </joint>
         <link name="gripper_scups_link">
-            <visual>
+            <!-- <visual>
                 <geometry>
                     <box size="0.01 0.01 0.01" />
@@ -15,5 +15,5 @@
                     <color rgba="0 1 0 1" />
                 </material>
-            </visual>
+            </visual> -->
         </link>
         <joint name="gripper_palm_camera_joint" type="fixed">
@@ -26,10 +26,9 @@
             <child link="gripper_top_camera_link" />
             <origin xyz="0.00 -.072 -0.0865" rpy="0 0 0" />
-            <!-- <origin xyz="0.009525 -.08255 -0.0445" rpy="0 0 0"/> -->
         </joint>
         <link name="gripper_top_camera_link">
         </link>
         <link name="gripper_palm_camera_optical_link">
-            <visual>
+            <!-- <visual>
                 <geometry>
                     <box size="0.03 0.03 0.01" />
@@ -38,5 +37,5 @@
                     <color rgba="0 1 0 1" />
                 </material>
-            </visual>
+            </visual> -->
         </link>
         <link name="gripper_link">

Commit message: verifies hardware transforms

File: harvest_hardware/robot_custom_hardware/urdf/amiga.urdf.xacro (robot description, xacro)
@@ -19,5 +19,5 @@
     <xacro:property name="amiga_collision_box2_z" value='0.25' />
     <xacro:property name="amiga_tool0_mount_rotation" value="0.0 0.0 ${pi / 4}"/>
-    <xacro:property name="amiga_tool0_mount_position" value="-0.225 0.323256 1.0"/>
+    <xacro:property name="amiga_tool0_mount_position" value="-0.092075 0.3048 1.04775"/>
     <!-- ================== -->
     <!--       Links        -->
@@ -32,22 +32,57 @@
             <material name="LightLightGrey"/>
         </visual>
-        <!-- <collision>
-            <origin rpy="0.0 0.0 0.0" xyz="0.0 0.0 ${amiga_collision_box0_z / 2}"/>
+        <!-- Linear Rail -->
+        <collision>
+            <origin rpy="0.0 0.0 0.0" xyz="0.0 0.29845 0.97"/>
             <geometry>
-                <box size="${amiga_collision_box0_x} ${amiga_collision_box0_y} ${amiga_collision_box0_z}"/>
+                <box size="1.2 0.2 0.15"/>
             </geometry>
         </collision>
+        <visual>
+            <origin rpy="0.0 0.0 0.0" xyz="0.0 0.29845 0.97"/>
+            <geometry>
+                <box size="1.2 0.2 0.15"/>
+            </geometry>
+        </visual>
+        <!-- Mast -->
         <collision>
-            <origin rpy="0.0 0.0 0.0" xyz="0.0 -${amiga_collision_box1_y / 5} ${amiga_collision_box0_z}" />
+            <origin rpy="0.0 0.0 0.0" xyz="0.57 -0.15 1.03"/>
             <geometry>
-                <box size="${amiga_collision_box1_x} ${amiga_collision_box1_y} ${amiga_collision_box1_z}" />
+                <box size="0.07 0.07 0.95"/>
             </geometry>
         </collision>
+        <visual>
+            <origin rpy="0.0 0.0 0.0" xyz="0.57 -0.15 1.03"/>
+            <geometry>
+                <box size="0.07 0.07 0.95"/>
+            </geometry>
+        </visual>
+        <!-- GPS & Oak cameras -->
         <collision>
-            <origin rpy="0.0 0.0 0.0" xyz="${amiga_collision_box0_x / 2 - amiga_collision_box2_x / 2} ${amiga_collision_box2_y / 3} ${amiga_collision_box0_z + amiga_collision_box1_z}" />
+            <origin rpy="0.0 0.0 0.0" xyz="0.57 -0.15 1.6"/>
             <geometry>
-                <box size="${amiga_collision_box2_x} ${amiga_collision_box2_y} ${amiga_collision_box2_z}" />
+                <box size="0.15 0.2 0.2"/>
             </geometry>
-        </collision> -->
+        </collision>
+        <visual>
+            <origin rpy="0.0 0.0 0.0" xyz="0.57 -0.15 1.6"/>
+            <geometry>
+                <box size="0.15 0.2 0.2"/>
+            </geometry>
+        </visual>
+        <!-- Amiga Brain -->
+        <collision>
+            <origin rpy="0.0 0.0 0.0" xyz="0.57 -0.315 1.25"/>
+            <geometry>
+                <box size="0.29 0.2 0.175"/>
+            </geometry>
+        </collision>
+        <visual>
+            <origin rpy="0.0 0.0 0.0" xyz="0.57 -0.315 1.25"/>
+            <geometry>
+                <box size="0.29 0.2 0.175"/>
+            </geometry>
+        </visual>
+        <!-- Base -->
         <collision>
             <origin rpy="0.0 0.0 0.0" xyz="0.0 0.0 0.0"/>

File: harvest_hardware/robot_custom_hardware/urdf/amiga_ur_gripper.urdf.xacro (robot description, xacro)
@@ -101,10 +101,10 @@
   </joint>
   <xacro:gripper_macro/>
-  <!-- Realsense for apple locations -->
+  <!-- MAST Realsense for apple locations -->
   <xacro:sensor_d435i
     parent="$(arg amiga_prefix)base"
     prefix="mast_"
     use_nominal_extrinsics="$(arg use_nominal_extrinsics)">
-    <origin xyz="0.3 -0.2 1.4667" rpy="0 0 1.8852"/>
+    <origin xyz="0.4064 -0.1778 1.5113" rpy="0 0 1.8852"/>
   </xacro:sensor_d435i>
   <!-- Realsense for trunk detections -->
@@ -113,5 +113,5 @@
     prefix="base_"
     use_nominal_extrinsics="$(arg use_nominal_extrinsics)">
-    <origin xyz="0.0 0.385 0.5588" rpy="0 0 1.57"/>
+    <origin xyz="0.0 0.3937 0.555625" rpy="0 0 1.57"/>
   </xacro:sensor_d435i>
 </robot>

Commit message: filters apple prediction relative to the cam position (left and right), and updates mast camera position

File: harvest_hardware/robot_custom_hardware/urdf/amiga.urdf.xacro (robot description, xacro)
@@ -19,5 +19,5 @@
     <xacro:property name="amiga_collision_box2_z" value='0.25' />
     <xacro:property name="amiga_tool0_mount_rotation" value="0.0 0.0 ${pi / 4}"/>
-    <xacro:property name="amiga_tool0_mount_position" value="-0.092075 0.3048 1.04775"/>
+    <xacro:property name="amiga_tool0_mount_position" value="-0.095 0.306 1.04775"/>
     <!-- ================== -->
     <!--       Links        -->

File: harvest_hardware/robot_custom_hardware/urdf/amiga_ur_gripper.urdf.xacro (robot description, xacro)
@@ -106,5 +106,9 @@
     prefix="mast_"
     use_nominal_extrinsics="$(arg use_nominal_extrinsics)">
-    <origin xyz="0.4064 -0.1778 1.5113" rpy="0 0 1.8852"/>
+    <!-- <origin xyz="0.4064 -0.1778 1.5113" rpy="0 0 1.8852"/> --> <!-- Manually measured position and orientation -->
+    <!-- <origin xyz="0.40948 -0.1881 1.5105" rpy="-0.013 0.033 1.907"/> Measured position and orientation with UR5e (with trailing values on roll and pitch -->
+    <!-- <origin xyz="0.40948 -0.1881 1.5105" rpy="0 0 1.907"/> Measured position and orientation with UR5e -->
+    <!-- <origin xyz="0.36566724 -0.17676987  1.52188824" rpy="-0.013000935978729311 0.03299973035765147 1.906999859790441"/> Calibrated from vision -->
+    <origin xyz=" 0.36916121 -0.17930941  1.534915" rpy="0 0 1.907"/>
   </xacro:sensor_d435i>
   <!-- Realsense for trunk detections -->
@@ -115,3 +119,20 @@
     <origin xyz="0.0 0.3937 0.555625" rpy="0 0 1.57"/>
   </xacro:sensor_d435i>
+  <!-- Tracking marker frame -->
+  <joint name="tracking_marker_joint" type="fixed">
+    <parent link="tool0"/>
+    <child  link="tool0_tracking_marking_link"/>
+    <origin xyz="0 0.12 0.037" rpy="0 0 0"/>
+  </joint>
+  <link name="tool0_tracking_marking_link">
+    <visual>
+      <origin xyz="0 0 0" rpy="0 0 0"/>
+      <geometry>
+        <sphere radius="0.001"/>
+      </geometry>
+      <material name="marker_material">
+        <color rgba="1 0 0 1"/>
+      </material>
+    </visual>
+  </link>
 </robot>
