Commit message: things are working in sim now sort of

File: harvest_hardware/robot_custom_hardware/urdf/amiga_ur_gripper.urdf.xacro (robot description, xacro)
@@ -103,12 +103,8 @@
   <!-- MAST Realsense for apple locations -->
   <xacro:sensor_d435i
-    parent="$(arg amiga_prefix)base"
+    parent="tool0"
     prefix="mast_"
     use_nominal_extrinsics="$(arg use_nominal_extrinsics)">
-    <!-- <origin xyz="0.4064 -0.1778 1.5113" rpy="0 0 1.8852"/> --> <!-- Manually measured position and orientation -->
-    <!-- <origin xyz="0.40948 -0.1881 1.5105" rpy="-0.013 0.033 1.907"/> Measured position and orientation with UR5e (with trailing values on roll and pitch -->
-    <!-- <origin xyz="0.40948 -0.1881 1.5105" rpy="0 0 1.907"/> Measured position and orientation with UR5e -->
-    <!-- <origin xyz="0.36566724 -0.17676987  1.52188824" rpy="-0.013000935978729311 0.03299973035765147 1.906999859790441"/> Calibrated from vision -->
-    <origin xyz=" 0.36916121 -0.17930941  1.534915" rpy="0 0 1.907"/>
+    <origin xyz="0.0 0.09 0.05" rpy="0 -1.57 -1.57"/>
   </xacro:sensor_d435i>
   <!-- Realsense for trunk detections -->

File: harvest_hardware/robot_custom_hardware/urdf/gripper.urdf.xacro (robot description, xacro)
@@ -40,21 +40,16 @@
         </link>
         <link name="gripper_link">
-            <collision>
-                <origin xyz="0.00 0 -0.105" rpy="0 0 0" />
-                <geometry>
-                    <box size="0.12 0.12 0.2" />
-                </geometry>
-            </collision>
-            <visual>
-                <origin xyz="0.085 0 -0.2" rpy="0 0 3.14" />
-                <geometry>
-                    <mesh
-                        filename="package://robot_custom_hardware/meshes/end_effectors/03_mk3_full_assembly_coarse.STL"
-                        scale="0.001 0.001 0.001" />
-                </geometry>
-                <material name="ur5_blue">
-                    <color rgba="0.45 0.62 0.9 1" />
-                </material>
-            </visual>
+        <collision>
+            <origin xyz="0 0 0" rpy="0 0 0" />
+            <geometry>
+            <cylinder radius="0.05" length="0.285" />
+            </geometry>
+        </collision>
+        <visual>
+            <origin xyz="0 0 0" rpy="0 0 0" />
+            <geometry>
+            <cylinder radius="0.05" length="0.285" />
+            </geometry>
+        </visual>
         </link>
     </xacro:macro>
