Commit message: restructure custom description and moveit config packages

File: harvest_hardware/harvest_hardware_description/urdf/amiga_ur_gripper.urdf.xacro (robot description, xacro)
@@ -2,5 +2,5 @@
 <robot xmlns:xacro="http://www.ros.org/wiki/xacro" name="$(arg name)">
   <!-- keep the basics -->
-  <xacro:arg name="name" default="ur"/>
+  <xacro:arg name="name" default="ur5e"/>
   <xacro:arg name="ur_type" default="ur5e"/>  <!-- absorbs CLI arg; we won't pass it to ur_robot -->
   <xacro:arg name="tf_prefix" default=""/>
@@ -33,29 +33,34 @@
   <xacro:arg name="sim_ignition" default="false"/>
   <xacro:arg name="simulation_controllers" default=""/>
-  <!-- initial positions in your pkg -->
-  <xacro:arg name="initial_positions_file" default="$(find robot_custom_hardware)/config/initial_positions.yaml"/>
+  <xacro:arg name="initial_positions_file" default="$(find harvest_hardware_description)/config/initial_positions.yaml"/>
   <xacro:property name="initial_positions_file" default="$(arg initial_positions_file)"/>
+  <!-- Amiga args -->
+  <xacro:arg name="amiga_prefix" default="amiga__"/>
   <!-- Realsense args -->
-  <xacro:arg name="use_nominal_extrinsics" default="false" />
-  <!-- CRITICAL: define the four args with the names the UR macro expects -->
-  <xacro:arg name="joint_limit_params" default="$(find robot_custom_hardware)/config/ur5e/joint_limits.yaml"/>
-  <xacro:arg name="kinematics_params"  default="$(find robot_custom_hardware)/config/ur5e/default_kinematics.yaml"/>
-  <xacro:arg name="physical_params"    default="$(find robot_custom_hardware)/config/ur5e/physical_parameters.yaml"/>
-  <xacro:arg name="visual_params"      default="$(find robot_custom_hardware)/config/ur5e/visual_parameters.yaml"/>
+  <xacro:arg name="use_nominal_extrinsics" default="true" />
+  <xacro:arg name="joint_limit_params" default="$(find ur_description)/config/$(arg ur_type)/joint_limits.yaml"/>
+  <xacro:arg name="kinematics_params" default="$(find ur_description)/config/$(arg ur_type)/default_kinematics.yaml"/>
+  <xacro:arg name="physical_params" default="$(find ur_description)/config/$(arg ur_type)/physical_parameters.yaml"/>
+  <xacro:arg name="visual_params" default="$(find ur_description)/config/$(arg ur_type)/visual_parameters.yaml"/>
   <!-- includes -->
+  <xacro:include filename="$(find harvest_hardware_description)/urdf/amiga.urdf.xacro"/>
   <xacro:include filename="$(find ur_description)/urdf/ur_macro.xacro"/>
-  <xacro:include filename="$(find robot_custom_hardware)/urdf/gripper.urdf.xacro"/>
-  <xacro:include filename="$(find realsense2_description)/urdf/_d435i.urdf.xacro"/>
+  <xacro:include filename="$(find harvest_hardware_description)/urdf/gripper.urdf.xacro"/>
+  <xacro:include filename="$(find harvest_hardware_description)/urdf/_d435i.urdf.xacro"/>
   <!-- define world exactly once -->
   <link name="world"/>
-  <!-- UR5e arm: DO NOT pass ur_type; just pass the four *_params -->
+  <!-- Instantiate Amiga, attached to world.
+       NOTE: your amiga macro signature requires mesh_base_path -->
+  <xacro:property name="harvest_hardware_description" value="package://harvest_hardware_description/"/>
+  <xacro:amiga_macro amiga_prefix="$(arg amiga_prefix)" amiga_parent="world" mesh_base_path="package://harvest_hardware_description/meshes/"/>
+  <!-- UR5e arm -->
   <xacro:ur_robot
       name="$(arg name)"
       tf_prefix="$(arg tf_prefix)"
-      parent="world"
-      joint_limits_parameters_file="$(arg joint_limit_params)"
-      kinematics_parameters_file ="$(arg kinematics_params)"
-      physical_parameters_file   ="$(arg physical_params)"
-      visual_parameters_file     ="$(arg visual_params)"
+      parent="$(arg amiga_prefix)tool0"
+      joint_limits_parameters_file="$(find ur_description)/config/$(arg ur_type)/joint_limits.yaml"
+      kinematics_parameters_file ="$(find ur_description)/config/$(arg ur_type)/default_kinematics.yaml"
+      physical_parameters_file   ="$(find ur_description)/config/$(arg ur_type)/physical_parameters.yaml"
+      visual_parameters_file     ="$(find ur_description)/config/$(arg ur_type)/visual_parameters.yaml"
       transmission_hw_interface="$(arg transmission_hw_interface)"
       safety_limits="$(arg safety_limits)"
@@ -95,6 +100,38 @@
   </joint>
   <xacro:gripper_macro/>
-  <xacro:sensor_d435i parent="base_link" use_nominal_extrinsics="$(arg use_nominal_extrinsics)">
-    <origin xyz="0.47625 -0.4907 0.4667" rpy="0 0 1.8852"/>
+  <!-- MAST Realsense for apple locations -->
+  <xacro:sensor_d435i
+    parent="$(arg amiga_prefix)base"
+    prefix="mast_"
+    use_nominal_extrinsics="$(arg use_nominal_extrinsics)">
+    <!-- <origin xyz="0.4064 -0.1778 1.5113" rpy="0 0 1.8852"/> --> <!-- Manually measured position and orientation -->
+    <!-- <origin xyz="0.40948 -0.1881 1.5105" rpy="-0.013 0.033 1.907"/> Measured position and orientation with UR5e (with trailing values on roll and pitch -->
+    <!-- <origin xyz="0.40948 -0.1881 1.5105" rpy="0 0 1.907"/> Measured position and orientation with UR5e -->
+    <!-- <origin xyz="0.36566724 -0.17676987  1.52188824" rpy="-0.013000935978729311 0.03299973035765147 1.906999859790441"/> Calibrated from vision -->
+    <origin xyz=" 0.36916121 -0.17930941  1.534915" rpy="0 0 1.907"/>
   </xacro:sensor_d435i>
+  <!-- Realsense for trunk detections -->
+  <xacro:sensor_d435i
+    parent="$(arg amiga_prefix)base"
+    prefix="base_"
+    use_nominal_extrinsics="$(arg use_nominal_extrinsics)">
+    <origin xyz="0.0 0.3937 0.555625" rpy="0 0 1.57"/>
+  </xacro:sensor_d435i>
+  <!-- Tracking marker frame -->
+  <joint name="tracking_marker_joint" type="fixed">
+    <parent link="tool0"/>
+    <child  link="tool0_tracking_marking_link"/>
+    <origin xyz="0 0.12 0.037" rpy="0 0 0"/>
+  </joint>
+  <link name="tool0_tracking_marking_link">
+    <visual>
+      <origin xyz="0 0 0" rpy="0 0 0"/>
+      <geometry>
+        <sphere radius="0.001"/>
+      </geometry>
+      <material name="marker_material">
+        <color rgba="1 0 0 1"/>
+      </material>
+    </visual>
+  </link>
 </robot>

File: harvest_hardware/harvest_hardware_description/urdf/gripper.urdf.xacro (robot description, xacro)
@@ -50,5 +50,5 @@
                 <geometry>
                     <mesh
-                        filename="package://robot_custom_hardware/meshes/end_effectors/03_mk3_full_assembly_coarse.STL"
+                        filename="package://harvest_hardware_description/meshes/end_effectors/03_mk3_full_assembly_coarse.STL"
                         scale="0.001 0.001 0.001" />
                 </geometry>

File: harvest_hardware/harvest_hardware_description/urdf/ur_gripper.urdf.xacro (robot description, xacro)
@@ -2,5 +2,5 @@
 <robot xmlns:xacro="http://www.ros.org/wiki/xacro" name="$(arg name)">
   <!-- keep the basics -->
-  <xacro:arg name="name" default="ur"/>
+  <xacro:arg name="name" default="ur5e"/>
   <xacro:arg name="ur_type" default="ur5e"/>  <!-- absorbs CLI arg; we won't pass it to ur_robot -->
   <xacro:arg name="tf_prefix" default=""/>
@@ -33,31 +33,25 @@
   <xacro:arg name="sim_ignition" default="false"/>
   <xacro:arg name="simulation_controllers" default=""/>
-  <xacro:arg name="initial_positions_file" default="$(find robot_custom_hardware)/config/initial_positions.yaml"/>
+  <!-- initial positions in your pkg -->
+  <xacro:arg name="initial_positions_file" default="$(find harvest_hardware_description)/config/initial_positions.yaml"/>
   <xacro:property name="initial_positions_file" default="$(arg initial_positions_file)"/>
-  <!-- Amiga args -->
-  <xacro:arg name="amiga_prefix" default="amiga__"/>
   <!-- Realsense args -->
-  <xacro:arg name="use_nominal_extrinsics" default="true" />
-  <!-- Define the four args with the names the UR macro expects -->
-  <xacro:arg name="joint_limit_params" default="$(find robot_custom_hardware)/config/ur5e/joint_limits.yaml"/>
-  <xacro:arg name="kinematics_params"  default="$(find robot_custom_hardware)/config/ur5e/default_kinematics.yaml"/>
-  <xacro:arg name="physical_params"    default="$(find robot_custom_hardware)/config/ur5e/physical_parameters.yaml"/>
-  <xacro:arg name="visual_params"      default="$(find robot_custom_hardware)/config/ur5e/visual_parameters.yaml"/>
+  <xacro:arg name="use_nominal_extrinsics" default="false" />
+  <!-- CRITICAL: define the four args with the names the UR macro expects -->
+  <xacro:arg name="joint_limit_params" default="$(find ur_description)/config/$(arg ur_type)/joint_limits.yaml"/>
+  <xacro:arg name="kinematics_params" default="$(find ur_description)/config/$(arg ur_type)/default_kinematics.yaml"/>
+  <xacro:arg name="physical_params" default="$(find ur_description)/config/$(arg ur_type)/physical_parameters.yaml"/>
+  <xacro:arg name="visual_params" default="$(find ur_description)/config/$(arg ur_type)/visual_parameters.yaml"/>
   <!-- includes -->
-  <xacro:include filename="$(find robot_custom_hardware)/urdf/amiga.urdf.xacro"/>
   <xacro:include filename="$(find ur_description)/urdf/ur_macro.xacro"/>
-  <xacro:include filename="$(find robot_custom_hardware)/urdf/gripper.urdf.xacro"/>
-  <xacro:include filename="$(find robot_custom_hardware)/urdf/_d435i.urdf.xacro"/>
+  <xacro:include filename="$(find harvest_hardware_description)/urdf/gripper.urdf.xacro"/>
+  <xacro:include filename="$(find realsense2_description)/urdf/_d435i.urdf.xacro"/>
   <!-- define world exactly once -->
   <link name="world"/>
-  <!-- Instantiate Amiga, attached to world.
-       NOTE: your amiga macro signature requires mesh_base_path -->
-  <xacro:property name="robot_custom_hardware" value="package://robot_custom_hardware/"/>
-  <xacro:amiga_macro amiga_prefix="$(arg amiga_prefix)" amiga_parent="world" mesh_base_path="package://robot_custom_hardware/meshes/"/>
-  <!-- UR5e arm -->
+  <!-- UR5e arm: DO NOT pass ur_type; just pass the four *_params -->
   <xacro:ur_robot
       name="$(arg name)"
       tf_prefix="$(arg tf_prefix)"
-      parent="$(arg amiga_prefix)tool0"
+      parent="world"
       joint_limits_parameters_file="$(arg joint_limit_params)"
       kinematics_parameters_file ="$(arg kinematics_params)"
@@ -101,38 +95,6 @@
   </joint>
   <xacro:gripper_macro/>
-  <!-- MAST Realsense for apple locations -->
-  <xacro:sensor_d435i
-    parent="$(arg amiga_prefix)base"
-    prefix="mast_"
-    use_nominal_extrinsics="$(arg use_nominal_extrinsics)">
-    <!-- <origin xyz="0.4064 -0.1778 1.5113" rpy="0 0 1.8852"/> --> <!-- Manually measured position and orientation -->
-    <!-- <origin xyz="0.40948 -0.1881 1.5105" rpy="-0.013 0.033 1.907"/> Measured position and orientation with UR5e (with trailing values on roll and pitch -->
-    <!-- <origin xyz="0.40948 -0.1881 1.5105" rpy="0 0 1.907"/> Measured position and orientation with UR5e -->
-    <!-- <origin xyz="0.36566724 -0.17676987  1.52188824" rpy="-0.013000935978729311 0.03299973035765147 1.906999859790441"/> Calibrated from vision -->
-    <origin xyz=" 0.36916121 -0.17930941  1.534915" rpy="0 0 1.907"/>
+  <xacro:sensor_d435i parent="base_link" use_nominal_extrinsics="$(arg use_nominal_extrinsics)">
+    <origin xyz="0.47625 -0.4907 0.4667" rpy="0 0 1.8852"/>
   </xacro:sensor_d435i>
-  <!-- Realsense for trunk detections -->
-  <xacro:sensor_d435i
-    parent="$(arg amiga_prefix)base"
-    prefix="base_"
-    use_nominal_extrinsics="$(arg use_nominal_extrinsics)">
-    <origin xyz="0.0 0.3937 0.555625" rpy="0 0 1.57"/>
-  </xacro:sensor_d435i>
-  <!-- Tracking marker frame -->
-  <joint name="tracking_marker_joint" type="fixed">
-    <parent link="tool0"/>
-    <child  link="tool0_tracking_marking_link"/>
-    <origin xyz="0 0.12 0.037" rpy="0 0 0"/>
-  </joint>
-  <link name="tool0_tracking_marking_link">
-    <visual>
-      <origin xyz="0 0 0" rpy="0 0 0"/>
-      <geometry>
-        <sphere radius="0.001"/>
-      </geometry>
-      <material name="marker_material">
-        <color rgba="1 0 0 1"/>
-      </material>
-    </visual>
-  </link>
 </robot>

Commit message: adds capability to view odometry or do regular motion planning

File: harvest_hardware/harvest_hardware_description/urdf/amiga_ur_gripper.urdf.xacro (robot description, xacro)
@@ -1,7 +1,7 @@
 <?xml version="1.0"?>
 <robot xmlns:xacro="http://www.ros.org/wiki/xacro" name="$(arg name)">
-  <!-- keep the basics -->
+  <!-- UR5e parameters -->
   <xacro:arg name="name" default="ur5e"/>
-  <xacro:arg name="ur_type" default="ur5e"/>  <!-- absorbs CLI arg; we won't pass it to ur_robot -->
+  <xacro:arg name="ur_type" default="ur5e"/>
   <xacro:arg name="tf_prefix" default=""/>
   <xacro:arg name="transmission_hw_interface" default=""/>
@@ -33,14 +33,15 @@
   <xacro:arg name="sim_ignition" default="false"/>
   <xacro:arg name="simulation_controllers" default=""/>
-  <xacro:arg name="initial_positions_file" default="$(find harvest_hardware_description)/config/initial_positions.yaml"/>
-  <xacro:property name="initial_positions_file" default="$(arg initial_positions_file)"/>
   <!-- Amiga args -->
   <xacro:arg name="amiga_prefix" default="amiga__"/>
   <!-- Realsense args -->
   <xacro:arg name="use_nominal_extrinsics" default="true" />
+  <!-- parameter files -->
   <xacro:arg name="joint_limit_params" default="$(find ur_description)/config/$(arg ur_type)/joint_limits.yaml"/>
   <xacro:arg name="kinematics_params" default="$(find ur_description)/config/$(arg ur_type)/default_kinematics.yaml"/>
   <xacro:arg name="physical_params" default="$(find ur_description)/config/$(arg ur_type)/physical_parameters.yaml"/>
   <xacro:arg name="visual_params" default="$(find ur_description)/config/$(arg ur_type)/visual_parameters.yaml"/>
+  <xacro:arg name="initial_positions_file" default="$(find harvest_hardware_description)/config/initial_positions.yaml"/>
+  <xacro:property name="initial_positions_file" default="$(arg initial_positions_file)"/>
   <!-- includes -->
   <xacro:include filename="$(find harvest_hardware_description)/urdf/amiga.urdf.xacro"/>
@@ -51,5 +52,5 @@
   <link name="world"/>
   <!-- Instantiate Amiga, attached to world.
-       NOTE: your amiga macro signature requires mesh_base_path -->
+       NOTE: the amiga macro signature requires mesh_base_path -->
   <xacro:property name="harvest_hardware_description" value="package://harvest_hardware_description/"/>
   <xacro:amiga_macro amiga_prefix="$(arg amiga_prefix)" amiga_parent="world" mesh_base_path="package://harvest_hardware_description/meshes/"/>
@@ -95,5 +96,5 @@
   <!-- mount gripper -->
   <joint name="gripper_joint" type="fixed">
-    <parent link="tool0"/>
+    <parent link="$(arg tf_prefix)tool0"/>
     <child  link="gripper_link"/>
     <origin xyz="0.00 0.00 0.215" rpy="0 0 0"/>
@@ -105,8 +106,4 @@
     prefix="mast_"
     use_nominal_extrinsics="$(arg use_nominal_extrinsics)">
-    <!-- <origin xyz="0.4064 -0.1778 1.5113" rpy="0 0 1.8852"/> --> <!-- Manually measured position and orientation -->
-    <!-- <origin xyz="0.40948 -0.1881 1.5105" rpy="-0.013 0.033 1.907"/> Measured position and orientation with UR5e (with trailing values on roll and pitch -->
-    <!-- <origin xyz="0.40948 -0.1881 1.5105" rpy="0 0 1.907"/> Measured position and orientation with UR5e -->
-    <!-- <origin xyz="0.36566724 -0.17676987  1.52188824" rpy="-0.013000935978729311 0.03299973035765147 1.906999859790441"/> Calibrated from vision -->
     <origin xyz=" 0.36916121 -0.17930941  1.534915" rpy="0 0 1.907"/>
   </xacro:sensor_d435i>
@@ -120,5 +117,5 @@
   <!-- Tracking marker frame -->
   <joint name="tracking_marker_joint" type="fixed">
-    <parent link="tool0"/>
+    <parent link="$(arg tf_prefix)tool0"/>
     <child  link="tool0_tracking_marking_link"/>
     <origin xyz="0 0.12 0.037" rpy="0 0 0"/>
