Commit message: trying to merge nicely...

File: harvest_hardware/harvest_hardware_description/urdf/amiga_ur_gripper.urdf.xacro (robot description, xacro)
@@ -94,17 +94,28 @@
     <origin xyz="0 0 0" rpy="0 0 0"/>
   </xacro:ur_robot>
-  <!-- mount gripper -->
+  <xacro:gripper_macro/>
+  <joint name="tool0_mimic" type="fixed">
+    <parent link="tool0"/>
+    <child  link="wrist_tool0"/>
+    <origin xyz="0.00 0.00 0.00" rpy="0 0 0"/>
+  </joint>
+  <!-- mount gripper ADDING 2 CM FOR CAMERA-->
   <joint name="gripper_joint" type="fixed">
     <parent link="$(arg tf_prefix)tool0"/>
     <child  link="gripper_link"/>
-    <origin xyz="0.00 0.00 0.215" rpy="0 0 0"/>
+    <origin xyz="0.00 0.00 0.25" rpy="0 0 0"/>
   </joint>
-  <xacro:gripper_macro/>
-  <!-- MAST Realsense for apple locations -->
+  <joint name="flex_tip_joint" type="fixed">
+      <parent link="tool0" />
+      <child link="flex_tip_link" />
+      <origin xyz="0.00 0.00 0.285" rpy="0 0 0" />
+  </joint>
+  <!-- MAST Realsense for apple locations (mounted on gripper) -->
   <xacro:sensor_d435i
-    parent="$(arg amiga_prefix)base"
+    parent="tool0"
     prefix="mast_"
     use_nominal_extrinsics="$(arg use_nominal_extrinsics)">
-    <origin xyz=" 0.36916121 -0.17930941  1.534915" rpy="0 0 1.907"/>
+    <!-- camera 9 cm down, ... cm forward from tool0 -->
+    <origin xyz="0.00 0.09 0.05" rpy="0 -1.5708 -1.5708"/>
   </xacro:sensor_d435i>
   <!-- Realsense for trunk detections -->

File: harvest_hardware/harvest_hardware_description/urdf/gripper.urdf.xacro (robot description, xacro)
@@ -2,11 +2,13 @@
 <robot xmlns:xacro="http://www.ros.org/wiki/xacro">
     <xacro:macro name="gripper_macro">
+        <link name="wrist_tool0">
+        </link>
         <joint name="gripper_scups_joint" type="fixed">
             <parent link="gripper_link" />
             <child link="gripper_scups_link" />
-            <origin xyz="0.00 0.00 -0.02" rpy="0 0 -2.618" />
+            <origin xyz="0.00 0.00 0.1" rpy="0 0 -2.618" />
         </joint>
         <link name="gripper_scups_link">
-            <!-- <visual>
+            <visual>
                 <geometry>
                     <box size="0.01 0.01 0.01" />
@@ -15,5 +17,5 @@
                     <color rgba="0 1 0 1" />
                 </material>
-            </visual> -->
+            </visual>
         </link>
         <joint name="gripper_palm_camera_joint" type="fixed">
@@ -26,8 +28,50 @@
             <child link="gripper_top_camera_link" />
             <origin xyz="0.00 -.072 -0.0865" rpy="0 0 0" />
+            <!-- <origin xyz="0.009525 -.08255 -0.0445" rpy="0 0 0"/> -->
         </joint>
         <link name="gripper_top_camera_link">
+            <!-- <collision>
+            <geometry>
+                <box size="0.08 0.05 0.01"/>
+            </geometry>
+        </collision> -->
         </link>
         <link name="gripper_palm_camera_optical_link">
+            <visual>
+                <geometry>
+                    <box size="0.03 0.03 0.01" />
+                </geometry>
+                <material name="green">
+                    <color rgba="0 1 0 1" />
+                </material>
+            </visual>
+        </link>
+        <link name="gripper_link">
+            <collision>
+                <origin xyz="0.00 0 -0.07" rpy="0 0 0" />
+                <geometry>
+                    <cylinder radius="0.05" length="0.25" />
+                </geometry>
+            </collision>
+            <visual>
+                <origin xyz="0 0 -0.07" rpy="0 0 0" />
+                <geometry>
+                    <cylinder radius="0.05" length="0.25" />
+                </geometry>
+                <material name="cylinder_color">
+                    <color rgba="1 0 0 0.5" />
+                </material>
+            </visual>
+        </link>
+        <link name="flex_tip_link">
+        </link>
+        <joint name="camera_joint" type="fixed">
+            <!-- <parent link="gripper_link" /> -->
+            <parent link="base_link" />
+            <child link="camera_link" />
+            <!-- <origin xyz="0.00 0.00 0.5" rpy="0 0 0" /> -->
+            <origin xyz="0.00 -0.1 0.5" rpy="-1.57079 0 0" />
+        </joint>
+        <link name="camera_link">
             <!-- <visual>
                 <geometry>
@@ -39,23 +83,10 @@
             </visual> -->
         </link>
-        <link name="gripper_link">
-            <collision>
-                <origin xyz="0.00 0 -0.105" rpy="0 0 0" />
-                <geometry>
-                    <box size="0.12 0.12 0.2" />
-                </geometry>
-            </collision>
-            <visual>
-                <origin xyz="0.085 0 -0.2" rpy="0 0 3.14" />
-                <geometry>
-                    <mesh
-                        filename="package://harvest_hardware_description/meshes/end_effectors/03_mk3_full_assembly_coarse.STL"
-                        scale="0.001 0.001 0.001" />
-                </geometry>
-                <material name="ur5_blue">
-                    <color rgba="0.45 0.62 0.9 1" />
-                </material>
-            </visual>
-        </link>
+        <!-- <xacro:arg name="use_nominal_extrinsics" default="false" />
+    <xacro:include filename="$(find realsense2_description)/urdf/_d435i.urdf.xacro"/>
+    <xacro:sensor_d435i parent="gripper_top_camera_link" use_nominal_extrinsics="$(arg
+        use_nominal_extrinsics)">
+      <origin xyz="0 0 -0.5" rpy="0 -1.571 1.571"/>
+    </xacro:sensor_d435i> -->
     </xacro:macro>
 </robot>

File: harvest_hardware/harvest_hardware_description/urdf/ur_gripper.urdf.xacro (robot description, xacro)
@@ -2,5 +2,5 @@
 <robot xmlns:xacro="http://www.ros.org/wiki/xacro" name="$(arg name)">
   <!-- keep the basics -->
-  <xacro:arg name="name" default="ur5e"/>
+  <xacro:arg name="name" default="ur"/>
   <xacro:arg name="ur_type" default="ur5e"/>  <!-- absorbs CLI arg; we won't pass it to ur_robot -->
   <xacro:arg name="tf_prefix" default=""/>
@@ -34,67 +34,86 @@
   <xacro:arg name="simulation_controllers" default=""/>
   <!-- initial positions in your pkg -->
-  <xacro:arg name="initial_positions_file" default="$(find harvest_hardware_description)/config/initial_positions.yaml"/>
+  <xacro:arg name="initial_positions_file" default="$(find robot_custom_hardware)/config/initial_positions.yaml"/>
   <xacro:property name="initial_positions_file" default="$(arg initial_positions_file)"/>
   <!-- Realsense args -->
   <xacro:arg name="use_nominal_extrinsics" default="false" />
   <!-- CRITICAL: define the four args with the names the UR macro expects -->
-  <xacro:arg name="joint_limit_params" default="$(find ur_description)/config/$(arg ur_type)/joint_limits.yaml"/>
-  <xacro:arg name="kinematics_params" default="$(find ur_description)/config/$(arg ur_type)/default_kinematics.yaml"/>
-  <xacro:arg name="physical_params" default="$(find ur_description)/config/$(arg ur_type)/physical_parameters.yaml"/>
-  <xacro:arg name="visual_params" default="$(find ur_description)/config/$(arg ur_type)/visual_parameters.yaml"/>
+  <xacro:arg name="joint_limit_params" default="$(find robot_custom_hardware)/config/ur5e/joint_limits.yaml"/>
+  <xacro:arg name="kinematics_params"  default="$(find robot_custom_hardware)/config/ur5e/default_kinematics.yaml"/>
+  <xacro:arg name="physical_params"    default="$(find robot_custom_hardware)/config/ur5e/physical_parameters.yaml"/>
+  <xacro:arg name="visual_params"      default="$(find robot_custom_hardware)/config/ur5e/visual_parameters.yaml"/>
   <!-- includes -->
   <xacro:include filename="$(find ur_description)/urdf/ur_macro.xacro"/>
-  <xacro:include filename="$(find harvest_hardware_description)/urdf/gripper.urdf.xacro"/>
+  <xacro:include filename="$(find robot_custom_hardware)/urdf/gripper.urdf.xacro"/>
   <xacro:include filename="$(find realsense2_description)/urdf/_d435i.urdf.xacro"/>
   <!-- define world exactly once -->
   <link name="world"/>
-  <!-- UR5e arm: DO NOT pass ur_type; just pass the four *_params -->
-  <xacro:ur_robot
-      name="$(arg name)"
-      tf_prefix="$(arg tf_prefix)"
-      parent="world"
-      joint_limits_parameters_file="$(arg joint_limit_params)"
-      kinematics_parameters_file ="$(arg kinematics_params)"
-      physical_parameters_file   ="$(arg physical_params)"
-      visual_parameters_file     ="$(arg visual_params)"
-      transmission_hw_interface="$(arg transmission_hw_interface)"
-      safety_limits="$(arg safety_limits)"
-      safety_pos_margin="$(arg safety_pos_margin)"
-      safety_k_position="$(arg safety_k_position)"
-      use_fake_hardware="$(arg use_fake_hardware)"
-      fake_sensor_commands="$(arg fake_sensor_commands)"
-      sim_gazebo ="$(arg sim_gazebo)"
-      sim_ignition ="$(arg sim_ignition)"
-      headless_mode="$(arg headless_mode)"
-      initial_positions="${xacro.load_yaml(initial_positions_file)}"
-      use_tool_communication="$(arg use_tool_communication)"
-      tool_voltage="$(arg tool_voltage)"
-      tool_parity="$(arg tool_parity)"
-      tool_baud_rate="$(arg tool_baud_rate)"
-      tool_stop_bits="$(arg tool_stop_bits)"
-      tool_rx_idle_chars="$(arg tool_rx_idle_chars)"
-      tool_tx_idle_chars="$(arg tool_tx_idle_chars)"
-      tool_device_name="$(arg tool_device_name)"
-      tool_tcp_port="$(arg tool_tcp_port)"
-      robot_ip="$(arg robot_ip)"
-      script_filename="$(arg script_filename)"
-      output_recipe_filename="$(arg output_recipe_filename)"
-      input_recipe_filename="$(arg input_recipe_filename)"
-      reverse_ip="$(arg reverse_ip)"
-      script_command_port="$(arg script_command_port)"
-      reverse_port="$(arg reverse_port)"
-      script_sender_port="$(arg script_sender_port)"
-      trajectory_port="$(arg trajectory_port)">
-    <origin xyz="0 0 0" rpy="0 0 0"/>
-  </xacro:ur_robot>
-  <!-- mount gripper -->
+   <!-- arm -->
+   <xacro:ur_robot
+     name="$(arg name)"
+     tf_prefix="$(arg tf_prefix)"
+     parent="world"
+     joint_limits_parameters_file="$(arg joint_limit_params)"
+     kinematics_parameters_file="$(arg kinematics_params)"
+     physical_parameters_file="$(arg physical_params)"
+     visual_parameters_file="$(arg visual_params)"
+     transmission_hw_interface="$(arg transmission_hw_interface)"
+     safety_limits="$(arg safety_limits)"
+     safety_pos_margin="$(arg safety_pos_margin)"
+     safety_k_position="$(arg safety_k_position)"
+     use_fake_hardware="$(arg use_fake_hardware)"
+     fake_sensor_commands="$(arg fake_sensor_commands)"
+     sim_gazebo="$(arg sim_gazebo)"
+     sim_ignition="$(arg sim_ignition)"
+     headless_mode="$(arg headless_mode)"
+     initial_positions="${xacro.load_yaml(initial_positions_file)}"
+     use_tool_communication="$(arg use_tool_communication)"
+     tool_voltage="$(arg tool_voltage)"
+     tool_parity="$(arg tool_parity)"
+     tool_baud_rate="$(arg tool_baud_rate)"
+     tool_stop_bits="$(arg tool_stop_bits)"
+     tool_rx_idle_chars="$(arg tool_rx_idle_chars)"
+     tool_tx_idle_chars="$(arg tool_tx_idle_chars)"
+     tool_device_name="$(arg tool_device_name)"
+     tool_tcp_port="$(arg tool_tcp_port)"
+     robot_ip="$(arg robot_ip)"
+     script_filename="$(arg script_filename)"
+     output_recipe_filename="$(arg output_recipe_filename)"
+     input_recipe_filename="$(arg input_recipe_filename)"
+     reverse_ip="$(arg reverse_ip)"
+     script_command_port="$(arg script_command_port)"
+     reverse_port="$(arg reverse_port)"
+     script_sender_port="$(arg script_sender_port)"
+     trajectory_port="$(arg trajectory_port)"
+     >
+     <origin xyz="0 0 0" rpy="0 0 0" />          <!-- position robot in the world -->
+   </xacro:ur_robot>
+   <xacro:if value="$(arg sim_gazebo)">
+    <!-- Gazebo plugins -->
+    <gazebo reference="world">
+    </gazebo>
+    <gazebo>
+      <plugin filename="libgazebo_ros2_control.so" name="gazebo_ros2_control">
+        <parameters>$(arg simulation_controllers)</parameters>
+      </plugin>
+    </gazebo>
+  </xacro:if>
+  <xacro:if value="$(arg sim_ignition)">
+    <!-- Gazebo plugins -->
+    <gazebo reference="world">
+    </gazebo>
+    <gazebo>
+      <plugin filename="libign_ros2_control-system.so" name="ign_ros2_control::IgnitionROS2ControlPlugin">
+        <parameters>$(arg simulation_controllers)</parameters>
+        <controller_manager_node_name>$(arg tf_prefix)controller_manager</controller_manager_node_name>
+      </plugin>
+    </gazebo>
+  </xacro:if>
   <joint name="gripper_joint" type="fixed">
-    <parent link="tool0"/>
-    <child  link="gripper_link"/>
-    <origin xyz="0.00 0.00 0.215" rpy="0 0 0"/>
+        <parent link="tool0"/>
+        <child link="gripper_link"/>
+        <origin xyz="0.00 0.00 0.215" rpy="0 0 0"/>
   </joint>
-  <xacro:gripper_macro/>
-  <xacro:sensor_d435i parent="base_link" use_nominal_extrinsics="$(arg use_nominal_extrinsics)">
-    <origin xyz="0.47625 -0.4907 0.4667" rpy="0 0 1.8852"/>
-  </xacro:sensor_d435i>
+  <xacro:include filename="gripper.urdf.xacro"/>
+  <xacro:gripper_macro />
 </robot>
